File: SAO-SecDSM-DC26.kicad_pcb (KiCad board)
At the start: 2 copper layers, 30.5 x 28.6 mm, 25 parts, among them P1 CONN_01X02, P2 CONN_01X02, P3 CONN_01X02, P4 CONN_01X02, P5 CONN_01X02, P6 CONN_01X02, U1 TPIC2810, X1 Badgelife_shitty_connector

Commit message: Rev1
Parts:
- added G***: LOGO, SAO-SecDSM-DC26:glider, B.Cu at (155.6, 92.6)
Routing:
- net Net-(D7-Pad1): track 8.73 -> 3.85 mm
- net Net-(D8-Pad1): track 18.8 -> 21.4 mm, vias 3 -> 1
- net GND: track 33.4 -> 34.9 mm
- net Net-(D6-Pad1): track 6.19 -> 7.37 mm
Other:
- board text added: "DC26"
- board text added: "REV1"
- board text added: "drahos"
