File: SAO-SecDSM-DC26.sch (KiCad schematic (older format))
At the start: 24 parts, among them P1 CONN_01X02, P2 CONN_01X02, P3 CONN_01X02, P4 CONN_01X02, P5 CONN_01X02, P6 CONN_01X02, U1 TPIC2810, X1 Badgelife_shitty_connector

Commit message: Added BoM
Parts:
- D8: footprint LEDs:LED_0805_HandSoldering -> LEDs:LED_0603_HandSoldering
Changed lines of the file:
@@
 F 0 "D8" H 9100 2950 50  0000 C CNN
 F 1 "LED" H 9100 2750 50  0000 C CNN
-F 2 "LEDs:LED_0805_HandSoldering" H 9100 2850 50  0001 C CNN
+F 2 "LEDs:LED_0603_HandSoldering" H 9100 2850 50  0001 C CNN
 F 3 "" H 9100 2850 50  0000 C CNN
 	1    9100 2850
